File: motor-drive-controller/hardware/kicad/gate-driver.kicad_sch (KiCad schematic)
At the start: 13 parts, among them U3 DRV83053PHP

Commit message: feat(hw09): add WAKE control signal
Parts:
- removed R20: 47k, Resistor_SMD:R_0603_1608Metric, symbol Device:R
- added C34: 1n, Capacitor_SMD:C_0603_1608Metric, symbol Device:C
- added NT1: NetTie_2, symbol Device:NetTie_2
- added R23: 10k, Resistor_SMD:R_0603_1608Metric, symbol Device:R
- U3: value DRV83053PHP -> DRV8305NPHP; Check_prices https://www.snapeda.com/parts/DRV83053PHP/Texas+Instruments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 -> (none); MP DRV83053PHP -> DRV8305NPHP; Purchase-URL https://www.snapeda.com/api/url_track_click_mouser/?unipart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 -> (none); SnapEDA_Link https://www.snapeda.com/parts/DRV83053PHP/Texas+Instruments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 -> (none)
Connections:
- net +3.3V: no longer C16.1, U3.48 (VREG)
- net EP: now also NT1.1; no longer C16.2, C17.2, C20.2, C23.2, C24.2, U3.14 (GND), U3.45 (GND)
- net at U3.42 (CP1L): now also C18.2; no longer C18.1
- net at U3.43 (CP1H): now also C18.1; no longer C18.2
- net WAKE renamed DRV.WAKE
- net DRV.WAKE: now also C34.1, R23.2
- new net +5V: R23.1
- new net GND: C16.2, C17.2, C20.2, C23.2, C24.2, C34.2, NT1.2, U3.14 (GND), U3.45 (GND)
- new net VDDA +3.3V: C16.1, U3.48 (VREG)
Other:
- moved on the sheet: C16, C18, C19

Commit message: fix(hw09): update footprint property for NetTie in gate driver schematic
Parts:
- NT1: footprint (none) -> NetTie:NetTie-2_SMD_Pad0.5mm
Changed lines of the file:
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@@
 			)
 		)
-		(property "Footprint" ""
+		(property "Footprint" "NetTie:NetTie-2_SMD_Pad0.5mm"
 			(at 148.59 165.1 0)
 			(hide yes)
