File: motor-drive-controller/hardware/kicad/mcu.kicad_sch (KiCad schematic)
At the start: 28 parts, among them J2 Conn_01x03_Pin, J3 JTAG, J4 J_HALL, SW1 SW_Push, U1 STM32F405RGT6, U2 CR2032, Y1 AAH-181-8.000MHZ

Commit message: feat(hw10): reset annotate schematic
Parts:
- renumbered C9 to C1, C11 to C10, C13 to C11, C15 to C13, C5 to C2, C6 to C4, C4 to C5, C8 to C6, C22 to C8, C10 to C9, J3 to J1, J4 to J2, J2 to J3, R14 to R1, R19 to R2, R13 to R3, R17 to R4, R18 to R5, R11 to R6

Commit message: feat(hw10): add  power LDO +5V --> +3.3V schema
Changed lines of the file:
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@@
 	)
 	(junction
-		(at 53.34 107.95)
-		(diameter 0)
-		(color 0 0 0 0)
-	)
-	(junction
 		(at 246.38 50.8)
 		(diameter 0)
@@
 	(wire
 		(pts
-			(xy 53.34 107.95) (xy 63.5 107.95)
+			(xy 40.64 107.95) (xy 63.5 107.95)
 		)
 		(stroke
@@
 	(wire
 		(pts
+			(xy 30.48 162.56) (xy 33.02 162.56)
+		)
+		(stroke
+			(width 0)
+			(type default)
+		)
+	)
+	(wire
+		(pts
 			(xy 240.03 44.45) (xy 240.03 50.8)
 		)
@@
 	(wire
 		(pts
-			(xy 53.34 102.87) (xy 53.34 107.95)
-		)
-		(stroke
-			(width 0)
-			(type default)
-		)
-	)
-	(wire
-		(pts
 			(xy 53.34 68.58) (xy 53.34 69.85)
 		)
@@
 	(wire
 		(pts
-			(xy 40.64 107.95) (xy 53.34 107.95)
-		)
-		(stroke
-			(width 0)
-			(type default)
-		)
-	)
-	(wire
-		(pts
 			(xy 54.61 125.73) (xy 63.5 125.73)
 		)
@@
 	(wire
 		(pts
-			(xy 30.48 162.56) (xy 33.02 162.56)
-		)
-		(stroke
-			(width 0)
-			(type default)
-		)
-	)
-	(wire
-		(pts
 			(xy 163.83 60.96) (xy 176.53 60.96)
 		)
@@
 					(unit 1)
 				)
-			)
-		)
-	)
-	(symbol
-		(lib_id "power:PWR_FLAG")
-		(at 53.34 102.87 0)
-		(unit 1)
-		(body_style 1)
-		(exclude_from_sim no)
-		(in_bom yes)
-		(on_board yes)
-		(in_pos_files yes)
-		(dnp no)
-		(fields_autoplaced yes)
-		(property "Reference" "#FLG01"
-			(at 53.34 100.965 0)
-			(hide yes)
-			(show_name no)
-			(do_not_autoplace no)
-			(effects
-				(font
-					(size 1.27 1.27)
-				)
-			)
-		)
-		(property "Value" "PWR_FLAG"
-			(at 53.34 97.79 0)
-			(show_name no)
-			(do_not_autoplace no)
-			(effects
-				(font
-					(size 1.27 1.27)
-				)
-			)
-		)
-		(property "Footprint" ""
-			(at 53.34 102.87 0)
-			(hide yes)
-			(show_name no)
-			(do_not_autoplace no)
-			(effects
-				(font
-					(size 1.27 1.27)
-				)
-			)
-		)
-		(property "Datasheet" ""
-			(at 53.34 102.87 0)
-			(hide yes)
-			(show_name no)
-			(do_not_autoplace no)
-			(effects
-				(font
-					(size 1.27 1.27)
-				)
-			)
-		)
-		(property "Description" "Special symbol for telling ERC where power comes from"
-			(at 53.34 102.87 0)
-			(hide yes)
-			(show_name no)
-			(do_not_autoplace no)
-			(effects
-				(font
-					(size 1.27 1.27)
-				)
-			)
-		)
-		(pin "1"
-		)
-		(instances
-			(project "motor-drive-controller"
-				(path "/b8e0307a-d356-4cd3-91c6-dd251b6e910b/194c8782-4fa9-42ae-9e6d-f27cf422e161"
-					(reference "#FLG01")
-					(unit 1)
-				)
